File: PK_MUV/Tech/Eagle files/PK_MUV_L1.brd (EAGLE design)
At the start: 13 x 26.5 mm, 4 parts, among them U1 WS2812

Commit message: Update tech
Parts:
- removed R1: (no value), microbuilder:1206
- removed U1: WS2812, SparkFun-LED:LED-TRICOLOR-5050-IC
- added LED1: WS2812B_5050N, adafruit:WS2812B-NARROW
- C1: value (none) -> 0.1u
- moved C1 0.75 mm to (6.71, 19.6), turned to 180 degrees
Connections:
- net BAT: now also LED1.1-VDD; no longer R1.1, R1.2, U1.3, U1.5
- net GND: now also LED1.3-GND; no longer U1.6
- net IN_LIGHT: now also LED1.4-DIN; no longer U1.2
- net OUT_LIGHT: now also LED1.2-DOUT; no longer U1.1
Routing:
- net BAT: track 34.3 -> 18.4 mm
- net GND: track 18.8 -> 29.2 mm
- net IN_LIGHT: track 13.3 -> 9.26 mm
- net OUT_LIGHT: track 13.0 -> 14.2 mm
Changed lines of the file:
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@@
 <setting verticaltext="up"/>
 </settings>
-<grid distance="1" unitdist="mm" unit="mm" style="lines" multiple="1" display="yes" altdistance="5" altunitdist="mil" altunit="mil"/>
+<grid distance="0.1" unitdist="mm" unit="mm" style="lines" multiple="1" display="yes" altdistance="5" altunitdist="mil" altunit="mil"/>
 <layers>
 <layer number="1" name="Top" color="4" fill="1" visible="yes" active="yes"/>
@@
 </autorouter>
 <elements>
-<element name="U1" library="SparkFun-LED" package="LED-TRICOLOR-5050-IC" value="WS2812" x="6.59" y="13.8" smashed="yes" rot="MR180">
-<attribute name="NAME" x="6.59" y="11.133" size="0.6096" layer="26" font="vector" ratio="20" rot="MR180" align="bottom-center"/>
-<attribute name="PROD_ID" value="DIO-11598" x="6.59" y="13.8" size="1.778" layer="28" rot="MR180" display="off"/>
-<attribute name="VALUE" x="7.59" y="16.467" size="0.6096" layer="28" font="vector" ratio="20" rot="MR180" align="top-center"/>
+<element name="C1" library="microbuilder" package="1206" value="0.1u" x="6.71" y="19.62" smashed="yes" rot="MR180">
+<attribute name="NAME" x="9.45" y="21.547" size="0.8128" layer="26" ratio="18" rot="MR180"/>
+<attribute name="VALUE" x="9.65" y="20.455" size="0.4064" layer="28" ratio="10" rot="MR180"/>
 </element>
-<element name="C1" library="microbuilder" package="1206" value="" x="6.59" y="18.88" smashed="yes" rot="MR0">
-<attribute name="NAME" x="9.05" y="20.753" size="0.8128" layer="26" ratio="18" rot="MR0"/>
-<attribute name="VALUE" x="4.05" y="18.245" size="0.4064" layer="28" ratio="10" rot="MR0"/>
+<element name="JP1" library="microbuilder" package="1X04_OVAL" value="" x="6.5" y="2.6" rot="R180"/>
+<element name="LED1" library="adafruit" package="WS2812B-NARROW" value="WS2812B_5050N" x="6.6" y="13.2" smashed="yes" rot="MR90">
+<attribute name="NAME" x="3.8875" y="10.0925" size="0.8128" layer="26" ratio="10" rot="MR0"/>
 </element>
-<element name="R1" library="microbuilder" package="1206" value="" x="3.9" y="9.2" rot="MR180"/>
-<element name="JP1" library="microbuilder" package="1X04_OVAL" value="" x="6.5" y="2.6" rot="R180"/>
 </elements>
 <signals>
 <signal name="BAT" class="1">
-<contactref element="U1" pad="5"/>
-<contactref element="U1" pad="3"/>
 <contactref element="C1" pad="1"/>
-<wire x1="8.35" y1="18.75" x2="8" y2="18.75" width="1" layer="16"/>
-<wire x1="10.975" y1="16.125" x2="8.35" y2="18.75" width="1" layer="16"/>
-<wire x1="10.975" y1="14.9" x2="10.975" y2="16.125" width="1" layer="16"/>
-<wire x1="9.925" y1="13.85" x2="10.975" y2="14.9" width="1" layer="16"/>
-<wire x1="9.05" y1="13.85" x2="9.925" y2="13.85" width="1" layer="16"/>
-<wire x1="8" y1="18.75" x2="7.99" y2="18.88" width="1" layer="16"/>
-<wire x1="9.05" y1="13.85" x2="8.99" y2="13.8" width="1" layer="16"/>
-<wire x1="4.15" y1="15.95" x2="4.15" y2="15.6" width="1" layer="16"/>
-<wire x1="3.45" y1="16.65" x2="4.15" y2="15.95" width="1" layer="16"/>
-<wire x1="3.45" y1="20.15" x2="3.45" y2="16.65" width="1" layer="16"/>
-<wire x1="4.15" y1="20.85" x2="3.45" y2="20.15" width="1" layer="16"/>
-<wire x1="6.25" y1="20.85" x2="4.15" y2="20.85" width="1" layer="16"/>
-<wire x1="7.825" y1="19.275" x2="6.25" y2="20.85" width="1" layer="16"/>
-<wire x1="4.15" y1="15.6" x2="4.19" y2="15.5" width="1" layer="16"/>
-<wire x1="7.825" y1="19.275" x2="7.99" y2="18.88" width="1" layer="16"/>
-<contactref element="R1" pad="1"/>
-<contactref element="R1" pad="2"/>
-<wire x1="5.64" y1="8.86" x2="5.3" y2="9.2" width="1" layer="16"/>
-<wire x1="2.5" y1="9.2" x2="2.5" y2="10.115075" width="1" layer="16"/>
-<wire x1="2.5" y1="10.115075" x2="1.525" y2="11.090075" width="1" layer="16"/>
-<wire x1="1.525" y1="11.090075" x2="1.525" y2="14.725" width="1" layer="16"/>
-<wire x1="1.525" y1="14.725" x2="3.45" y2="16.65" width="1" layer="16"/>
 <contactref element="JP1" pad="3"/>
-<wire x1="5.3" y1="9.2" x2="5.3" y2="2.67" width="1" layer="16"/>
-<wire x1="5.3" y1="2.67" x2="5.23" y2="2.6" width="1" layer="16"/>
-<wire x1="5.3" y1="9.2" x2="2.5" y2="9.2" width="0" layer="19" extent="16-16"/>
+<contactref element="LED1" pad="1-VDD"/>
+<wire x1="5.075" y1="19.425" x2="5.075" y2="15.575" width="1" layer="16"/>
+<wire x1="5.25" y1="19.6" x2="5.075" y2="19.425" width="1" layer="16"/>
+<wire x1="5.075" y1="15.575" x2="4.95" y2="15.55" width="1" layer="16"/>
+<wire x1="5.25" y1="19.6" x2="5.31" y2="19.62" width="1" layer="16"/>
+<wire x1="5.25" y1="7.7" x2="5.25" y2="2.625" width="1" layer="16"/>
+<wire x1="6.475" y1="8.925" x2="5.25" y2="7.7" width="1" layer="16"/>
+<wire x1="6.475" y1="11.9" x2="6.475" y2="8.925" width="1" layer="16"/>
+<wire x1="4.9" y1="13.475" x2="6.475" y2="11.9" width="1" layer="16"/>
+<wire x1="4.9" y1="15.05" x2="4.9" y2="13.475" width="1" layer="16"/>
+<wire x1="5.25" y1="2.625" x2="5.23" y2="2.6" width="1" layer="16"/>
+<wire x1="4.9" y1="15.05" x2="4.95" y2="15.55" width="1" layer="16"/>
 </signal>
 <signal name="IN_LIGHT">
-<contactref element="U1" pad="2" route="any" routetag="U1.DI"/>
-<wire x1="3.625" y1="13.675" x2="4.15" y2="13.675" width="0.3" layer="16"/>
-<wire x1="3.625" y1="13.675" x2="2.575" y2="12.625" width="0.3" layer="16"/>
-<wire x1="4.15" y1="13.675" x2="4.19" y2="13.8" width="0.3" layer="16"/>
-<wire x1="2.575" y1="12.625" x2="2.575" y2="11.525" width="0.3" layer="16"/>
-<wire x1="2.575" y1="11.525" x2="3.15" y2="10.95" width="0.3" layer="16"/>
-<wire x1="3.15" y1="10.95" x2="3.22781875" y2="10.95" width="0.3" layer="16"/>
-<wire x1="3.22781875" y1="10.95" x2="3.85" y2="10.32781875" width="0.3" layer="16"/>
-<wire x1="3.85" y1="10.32781875" x2="3.85" y2="9.85" width="0.3" layer="16"/>
-<wire x1="3.85" y1="9.85" x2="3.9" y2="9.8" width="0.3" layer="16"/>
-<wire x1="3.9" y1="9.8" x2="3.9" y2="9.2" width="0.3" layer="16"/>
-<wire x1="3.9" y1="9.2" x2="3.9" y2="5.82" width="0.3" layer="16"/>
 <contactref element="JP1" pad="4"/>
-<wire x1="3.9" y1="5.82" x2="2.69" y2="4.61" width="0.3" layer="16"/>
-<wire x1="2.69" y1="4.61" x2="2.69" y2="2.6" width="0.3" layer="16"/>
+<contactref element="LED1" pad="4-DIN"/>
+<wire x1="4.9" y1="8.925" x2="4.9" y2="10.85" width="0.3" layer="16"/>
+<wire x1="2.8" y1="6.825" x2="4.9" y2="8.925" width="0.3" layer="16"/>
+<wire x1="2.8" y1="2.625" x2="2.8" y2="6.825" width="0.3" layer="16"/>
+<wire x1="4.9" y1="10.85" x2="4.95" y2="10.85" width="0.3" layer="16"/>
+<wire x1="2.8" y1="2.625" x2="2.69" y2="2.6" width="0.3" layer="16"/>
 </signal>
 <signal name="GND" class="1">
-<contactref element="U1" pad="6"/>
 <contactref element="C1" pad="2"/>
-<wire x1="5.2" y1="17" x2="5.2" y2="18.75" width="1" layer="16"/>
-<wire x1="6.95" y1="15.25" x2="5.2" y2="17" width="1" layer="16"/>
-<wire x1="6.95" y1="13.325" x2="6.95" y2="15.25" width="1" layer="16"/>
-<wire x1="8.175" y1="12.1" x2="6.95" y2="13.325" width="1" layer="16"/>
-<wire x1="8.875" y1="12.1" x2="8.175" y2="12.1" width="1" layer="16"/>
-<wire x1="5.2" y1="18.75" x2="5.19" y2="18.88" width="1" layer="16"/>
-<wire x1="8.875" y1="12.1" x2="8.99" y2="12.1" width="1" layer="16"/>
-<wire x1="10.1" y1="10.875" x2="10.1" y2="5.975" width="1" layer="16"/>
-<wire x1="9.225" y1="11.75" x2="10.1" y2="10.875" width="1" layer="16"/>
-<wire x1="9.225" y1="11.75" x2="8.99" y2="12.1" width="1" layer="16"/>
 <contactref element="JP1" pad="1"/>
-<wire x1="10.1" y1="5.975" x2="10.31" y2="5.765" width="1" layer="16"/>
-<wire x1="10.31" y1="5.765" x2="10.31" y2="2.6" width="1" layer="16"/>
+<contactref element="LED1" pad="3-GND"/>
+<wire x1="8.225" y1="12.25" x2="8.225" y2="10.85" width="1" layer="16"/>
+<wire x1="6.65" y1="13.825" x2="8.225" y2="12.25" width="1" layer="16"/>
+<wire x1="6.65" y1="13.825" x2="6.65" y2="16.95" width="1" layer="16"/>
+<wire x1="8.225" y1="10.85" x2="8.25" y2="10.85" width="1" layer="16"/>
+<wire x1="10.325" y1="3.675" x2="10.325" y2="2.625" width="1" layer="16"/>
+<wire x1="10.5" y1="3.85" x2="10.325" y2="3.675" width="1" layer="16"/>
+<wire x1="10.325" y1="2.625" x2="10.31" y2="2.6" width="1" layer="16"/>
+<wire x1="8.11" y1="19.62" x2="9.38" y2="19.62" width="1" layer="16"/>
+<wire x1="9.38" y1="19.62" x2="10.5" y2="18.5" width="1" layer="16"/>
+<wire x1="10.5" y1="18.5" x2="10.5" y2="3.85" width="1" layer="16"/>
+<wire x1="6.65" y1="16.95" x2="7.3" y2="17.6" width="1" layer="16"/>
+<wire x1="7.3" y1="17.6" x2="7.9" y2="17.6" width="1" layer="16"/>
+<wire x1="7.9" y1="17.6" x2="8.11" y2="17.81" width="1" layer="16"/>
+<wire x1="8.11" y1="17.81" x2="8.11" y2="19.62" width="1" layer="16"/>
 </signal>
 <signal name="OUT_LIGHT">
-<contactref element="U1" pad="1"/>
-<wire x1="4.59" y1="11.7" x2="4.19" y2="12.1" width="0.3" layer="16"/>
-<wire x1="6.2" y1="12" x2="8.18" y2="10.02" width="0.3" layer="16"/>
-<wire x1="6.2" y1="12" x2="4.29" y2="12" width="0.3" layer="16"/>
-<wire x1="4.29" y1="12" x2="4.19" y2="12.1" width="0.3" layer="16"/>
 <contactref element="JP1" pad="2"/>
-<wire x1="8.18" y1="10.02" x2="8.18" y2="3.01" width="0.3" layer="16"/>
-<wire x1="8.18" y1="3.01" x2="7.77" y2="2.6" width="0.3" layer="16"/>
+<contactref element="LED1" pad="2-DOUT"/>
+<wire x1="8.4" y1="13.65" x2="8.4" y2="15.4" width="0.3" layer="16"/>
+<wire x1="9.45" y1="12.6" x2="8.4" y2="13.65" width="0.3" layer="16"/>
+<wire x1="9.45" y1="4.375" x2="9.45" y2="12.6" width="0.3" layer="16"/>
+<wire x1="7.7" y1="2.625" x2="9.45" y2="4.375" width="0.3" layer="16"/>
+<wire x1="8.4" y1="15.4" x2="8.25" y2="15.55" width="0.3" layer="16"/>
+<wire x1="7.7" y1="2.625" x2="7.77" y2="2.6" width="0.3" layer="16"/>
 </signal>
 </signals>
