File: PK_MUV/Tech/Eagle files/PK_MUV_L2.brd (EAGLE design)
At the start: 28.1 x 21.3 mm, 6 parts, among them U1 WS2812, U2 WS2812

Commit message: Update tech
Parts:
- removed R1: 0, microbuilder:1206
- removed U1, U2: WS2812, SparkFun-LED:LED-TRICOLOR-5050-IC
- added LED1, LED2: WS2812B_5050N, adafruit:WS2812B-NARROW
- C1, C2: value (none) -> 0.1u
Connections:
- removed net N$1: JP1.2, U1.2
- removed net N$2: U1.1, U2.2
- new net IN: JP1.2, LED1.4-DIN
- new net N$3: LED1.2-DOUT, LED2.4-DIN
- new net VDD: LED2.1-VDD
- net BAT: now also LED1.1-VDD; no longer U1.3, U1.5, U2.3, U2.5
- net GND: now also LED1.3-GND, LED2.3-GND; no longer R1.1, R1.2, U1.6, U2.6
Routing:
- net BAT: track 74.3 -> 38.0 mm
- net N$3: track 0.00 -> 19.9 mm
- net N$1: track 18.2 -> 0.00 mm
- net N$2: track 16.5 -> 0.00 mm
- net IN: track 0.00 -> 8.80 mm
- net GND: track 48.4 -> 55.3 mm
Other:
- outline, holes or cut-outs redrawn
